File: hardware/sensor.sch (KiCad schematic (older format))
At the start: 56 parts, among them P1 CONN_01X05, SW1 Reset, T1 BUK9Y22, U1 LMR16006, U2 CD74HC4046, U3 CD74HC4046, U4 Atmel_SAM_D09, U5 OPA376AIDCK, X1 UART, X2 60V

Commit message: Fixed some schematic mistakes and footprints. Continued placing parts.
Parts:
- removed JP2_RX1: R_Small, Resistors_SMD:R_0603, symbol R_Small
- D_BLUE1, D_RED1: footprint Resistors_SMD:R_0603 -> LEDs:LED-0603
- R1: value R_Small -> 10k; footprint LEDs:LED_0603 -> Resistors_SMD:R_0603
- R1_RX1: footprint LEDs:LED_0603 -> Resistors_SMD:R_0603
Changed lines of the file:
@@
 F 0 "R1_RX1" V 3775 6600 50  0000 L CNN
 F 1 "R_Small" V 3625 6600 50  0000 L CNN
-F 2 "LEDs:LED_0603" H 3700 6675 50  0001 C CNN
+F 2 "Resistors_SMD:R_0603" H 3700 6675 50  0001 C CNN
 F 3 "" H 3700 6675 50  0000 C CNN
 	1    3700 6675
@@
 	1    0    0    -1
 $EndComp
-Text Label 2500 6550 2    60   ~ 0
+Text Label 2500 6525 2    60   ~ 0
 VCOin
 Text Label 5375 5350 2    60   ~ 0
 VCOin
-$Comp
-L R_Small JP2_RX1
-U 1 1 56E062DF
-P 5100 6425
-F 0 "JP2_RX1" V 5175 6350 50  0000 L CNN
-F 1 "R_Small" V 5025 6350 50  0001 L CNN
-F 2 "Resistors_SMD:R_0603" H 5100 6425 50  0001 C CNN
-F 3 "" H 5100 6425 50  0000 C CNN
-	1    5100 6425
-	0    1    1    0
-$EndComp
-Text Label 5475 6425 2    60   ~ 0
+Text Label 5275 6425 2    60   ~ 0
 JP2
 Text Label 3900 6025 2    60   ~ 0
@@
 F 0 "D_BLUE1" H 10175 2700 50  0000 L CNN
 F 1 "BLUE" H 10200 2475 50  0001 L CNN
-F 2 "Resistors_SMD:R_0603" V 10300 2575 50  0001 C CNN
+F 2 "LEDs:LED-0603" V 10300 2575 50  0001 C CNN
 F 3 "" V 10300 2575 50  0000 C CNN
 	1    10300 2575
@@
 F 0 "D_RED1" H 9850 2700 50  0000 L CNN
 F 1 "RED" H 9875 2475 50  0001 L CNN
-F 2 "Resistors_SMD:R_0603" V 9950 2575 50  0001 C CNN
+F 2 "LEDs:LED-0603" V 9950 2575 50  0001 C CNN
 F 3 "" V 9950 2575 50  0000 C CNN
 	1    9950 2575
@@
 P 6475 1950
 F 0 "R1" H 6505 1970 50  0000 L CNN
-F 1 "R_Small" H 6505 1910 50  0000 L CNN
-F 2 "LEDs:LED_0603" H 6475 1950 50  0001 C CNN
+F 1 "10k" H 6505 1910 50  0000 L CNN
+F 2 "Resistors_SMD:R_0603" H 6475 1950 50  0001 C CNN
 F 3 "" H 6475 1950 50  0000 C CNN
 	1    6475 1950
@@
 	3600 6875 3450 6875
 Wire Wire Line
-	5200 6425 5475 6425
+	5000 6425 5275 6425
 Wire Wire Line
 	5375 5350 5375 5500
@@
 	5350 475  5350 4800
 Connection ~ 1725 1275
+$Comp
+L GND #PWR032
+U 1 1 56E6FEBD
+P 1050 5525
+F 0 "#PWR032" H 1050 5275 50  0001 C CNN
+F 1 "GND" H 1050 5375 50  0000 C CNN
+F 2 "" H 1050 5525 50  0000 C CNN
+F 3 "" H 1050 5525 50  0000 C CNN
+	1    1050 5525
+	1    0    0    -1
+$EndComp
 $EndSCHEMATC
