File: hardware/_saved_sensor.sch (KiCad schematic (older format))
At the start: 55 parts, among them P1 CONN_01X05, SW1 Reset, T1 BUK9Y22, U1 LMR16006, U2 CD74HC4046, U3 CD74HC4046, U4 Atmel_SAM_D09, U5 OPA376AIDCK, X1 UART, X2 60V

Commit message: Finished placing for now
Parts:
- P1: footprint Pin_Headers:Pin_Header_Angled_1x05 -> Connectors_Molex:Connector_Molex_PicoBlade_53261-0571
Changed lines of the file:
@@
 F 0 "P1" H 6500 3150 50  0000 C CNN
 F 1 "CONN_01X05" V 6600 2850 50  0000 C CNN
-F 2 "Pin_Headers:Pin_Header_Angled_1x05" H 6500 2850 50  0001 C CNN
+F 2 "Connectors_Molex:Connector_Molex_PicoBlade_53261-0571" H 6500 2850 50  0001 C CNN
 F 3 "" H 6500 2850 50  0000 C CNN
 	1    6500 2850
