File: hardware/supervisor/supervisor.kicad_pcb (KiCad board)
At the start: 2 copper layers, 110 parts, among them IC1 ULN2003A, IC2 LM2596-3.3, IC3 MAX11612, IC4 ACS723LLCTR-10AU-T, IC5 ACS723LLCTR-10AU-T, IC6 ACS723LLCTR-10AU-T, IC7 NLSX4373, IC8 NLSX4373, IC9 SIM900, K1 RELAY_SERIE_36, K2 RELAY_SERIE_36, P1 230V_IN, P10 CONN_01X03, P11 CONN_01X03, P12 CONN_01X03, P13 230V_OUT, P14 230V_OUT, P15 230V_OUT, P2 RASPI-CONNECT, P3 POWER, P4 CONN_01X03, P5 230V_OUT, P6 CONN_01X03, P7 CONN_01X03, P8 CONN_01X03, P9 CONN_01X03, SW1 SW_PUSH, SW2 SW_PUSH, U1 SC16IS740IPW, U10 OPA376AIDCK, U11 CD74HC4046, U12 OPA376AIDCK, U16 CD74HC4046, U17 OPA376AIDCK, U2 SC16IS740IPW, U3 SC16IS740IPW, U4 RF_CONN, U5 SIM_HOLDER, U9 CD74HC4046

Commit message: routing 0.1
Parts:
- C20, C22, C23, C24, C26, C28, C29, C30, C43, C45, C46, C47, D6, D7, D8, R23, R24, R25, R26, R27, R28, R29, R30, R31, R32, R33, R34, R35, R36, R37, R38, R39, R54, R55, R56, R57, R58, R59, R60, R61, R62, U10, U11, U12, U16, U17, U2, U9: moved to B.Cu
- C6, C7, IC9, R5, R6, R7, U4, U5: moved to F.Cu
- moved C28 237.9 mm to (74.6, 58.2), turned to 180 degrees
- moved R36 229.1 mm to (79.6, 60.0), turned to 90 degrees
- moved R27 213.5 mm to (100.8, 53.7)
- moved C21 187.6 mm to (100.1, 124.7)
- moved C27 187.6 mm to (100.1, 127.3)
- moved C3 187.6 mm to (105.4, 109.7)
- moved C4 187.6 mm to (105.7, 112.3)
- moved C5 187.6 mm to (105.4, 118.6)
- moved C44 187.6 mm to (99.8, 99.8)
- moved R61 155.8 mm to (49.5, 49.3), turned to 180 degrees
- moved R59 153.0 mm to (46.7, 51.8), turned to 0 degrees
- moved C45 151.6 mm to (46.7, 53.7), turned to 180 degrees
- moved R60 151.4 mm to (52.8, 49.3), turned to 180 degrees
- moved C47 150.8 mm to (60.2, 49.3)
- moved R62 150.7 mm to (56.7, 49.3)
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Routing:
- net +5V: track 0.00 -> 222.9 mm, vias 0 -> 3
- net +3V3: track 0.00 -> 118.5 mm, vias 0 -> 1
- net Net-(IC1-Pad12): track 0.00 -> 99.3 mm, vias 0 -> 2
- net Net-(IC1-Pad11): track 0.00 -> 85.6 mm, vias 0 -> 2
- net GSM_LED0: track 0.00 -> 82.5 mm
- net GSM_PKEY: track 0.00 -> 82.1 mm
- net GSM_LED1: track 0.00 -> 65.8 mm
- net Net-(C6-Pad1): track 0.00 -> 61.9 mm
- net Net-(IC9-Pad60): track 0.00 -> 49.3 mm
- net ENSK0: track 0.00 -> 46.8 mm, vias 0 -> 1
- net RXD: track 0.00 -> 44.3 mm
- net Net-(D5-Pad1): track 0.00 -> 41.2 mm
- net TXD: track 0.00 -> 40.5 mm
- net Net-(C7-Pad1): track 0.00 -> 34.3 mm, vias 0 -> 2
- net Net-(K1-Pad14): track 0.00 -> 30.6 mm
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
Commit message: routing 0.2
Parts:
- moved D6 2.63 mm to (90.3, 59.4)
- moved C30 2.27 mm to (74.6, 49.8), turned to 0 degrees
- moved RV3 1.95 mm to (93.0, 56.9)
- moved C28 1.92 mm to (76.5, 57.7), turned to 90 degrees
- moved R31 1.63 mm to (74.6, 52.8)
- moved C26 1.38 mm to (74.5, 55.1)
- moved SW1 0.87 mm to (5.84, 42.2)
- moved SW2 0.87 mm to (5.84, 34.8)
- moved R54 0.65 mm to (62.4, 62.5)
- moved R23 0.51 mm to (102.1, 60.5)
- moved R25 0.51 mm to (96.4, 60.4)
- moved R29 0.51 mm to (98.3, 60.4)
- moved R28 0.51 mm to (100.3, 60.5)
Routing:
- net +3V3: track 118.5 -> 294.3 mm, vias 1 -> 7
- net SDA: track 14.9 -> 143.8 mm, vias 0 -> 5
- net +5V: track 222.9 -> 351.0 mm, vias 3 -> 6
- net ENSK2: track 0.00 -> 115.3 mm, vias 0 -> 2
- net MUCLK: track 0.00 -> 84.6 mm, vias 0 -> 3
- net SCL: track 16.9 -> 99.9 mm, vias 0 -> 4
- net GND: track 0.00 -> 82.4 mm, vias 0 -> 24
- net ENSK1: track 0.00 -> 70.5 mm
- net IRQ2: track 0.00 -> 59.0 mm, vias 0 -> 2
- net IRQ1: track 0.00 -> 33.6 mm, vias 0 -> 2
- net IRQ0: track 0.00 -> 21.1 mm, vias 0 -> 1
- net Net-(C43-Pad1): track 2.48 -> 18.4 mm
- net Net-(C20-Pad1): track 10.4 -> 25.7 mm, vias 0 -> 1
- net Net-(C26-Pad1): track 6.84 -> 21.1 mm
- net /FSK Module 1/incoming1: track 2.77 -> 14.9 mm, vias 0 -> 1
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Other:
- net class 0.4: clearance 0.25 -> 0.2
- net class Default: clearance 0.25 -> 0.2
- rule trace_clearance: 0.25 -> 0.2
