File: hardware/supervisor/supervisor.kicad_pcb (KiCad board)
At the start: 2 copper layers, 110 parts, among them IC1 ULN2003A, IC2 LM2596-3.3, IC3 MAX11612, IC4 ACS723LLCTR-10AU-T, IC5 ACS723LLCTR-10AU-T, IC6 ACS723LLCTR-10AU-T, IC7 NLSX4373, IC8 NLSX4373, IC9 SIM900, K1 RELAY_SERIE_36, K2 RELAY_SERIE_36, P1 230V_IN, P10 CONN_01X03, P11 CONN_01X03, P12 CONN_01X03, P13 230V_OUT, P14 230V_OUT, P15 230V_OUT, P2 RASPI-CONNECT, P3 POWER, P4 CONN_01X03, P5 230V_OUT, P6 CONN_01X03, P7 CONN_01X03, P8 CONN_01X03, P9 CONN_01X03, SW1 SW_PUSH, SW2 SW_PUSH, U1 SC16IS740IPW, U10 OPA376AIDCK, U11 CD74HC4046, U12 OPA376AIDCK, U16 CD74HC4046, U17 OPA376AIDCK, U2 SC16IS740IPW, U3 SC16IS740IPW, U4 RF_CONN, U5 SIM_HOLDER, U9 CD74HC4046

Commit message: routing 1.0 to review
Parts:
- C21, C27, C44: moved to B.Cu
- moved C5 75.0 mm to (56.0, 62.2), turned to 90 degrees
- moved C21 53.6 mm to (80.5, 74.8), turned to 180 degrees
- moved C27 52.5 mm to (98.8, 74.8)
- moved C3 49.0 mm to (78.1, 69.0)
- moved C44 44.9 mm to (62.5, 74.9), turned to 180 degrees
- moved C4 43.6 mm to (99.3, 69.2)
- moved P5 8.76 mm to (17.4, 5.99), turned to 0 degrees
- moved P4 5.57 mm to (30.5, 79.5)
- moved P6 5.14 mm to (62.3, 79.5)
- moved P7 5.02 mm to (77.6, 79.5)
- moved P8 4.86 mm to (92.8, 79.5)
- moved P12 4.23 mm to (10.2, 79.5)
- moved P1 3.08 mm to (7.62, 7.00)
- moved P9 1.06 mm to (87.1, 68.1)
Routing:
- net GND: track 82.4 -> 174.2 mm, vias 24 -> 40
- net Net-(P1-Pad1): track 0.00 -> 15.9 mm
- net PGND0: track 10.9 -> 22.3 mm
- net SCL: track 99.9 -> 88.5 mm, vias 4 -> 5
- net Net-(P13-Pad1): track 2.22 -> 12.0 mm
- net Net-(P14-Pad1): track 0.00 -> 9.30 mm
- net Net-(IC8-Pad8): track 20.0 -> 28.0 mm
- net string_out1: track 1.28 -> 9.20 mm
- net +3V3: track 294.3 -> 302.1 mm, vias 7 -> 11
- net Net-(P1-Pad2): track 0.00 -> 7.63 mm
- net string_out2: track 1.27 -> 8.41 mm
- net string_out0: track 4.05 -> 10.9 mm
- net PGND1: track 7.73 -> 13.7 mm
- net PGND2: track 12.0 -> 17.5 mm
- net Net-(K2-Pad14): track 29.9 -> 25.7 mm
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Other:
- board text added: "Supervisor v1.0 altyr 2016"

Commit message: routing 1.1 to release
Parts:
- moved U4 1.76 mm to (98.3, 4.72)
Routing:
- net GND: track 174.2 -> 160.2 mm, vias 40 -> 32
- net (no net): track 0.00 -> 14.0 mm, vias 0 -> 8
- net Net-(IC9-Pad60): track 49.3 -> 48.7 mm
Other:
- board text added: "Supervisor v1.1 altyr 2016"
- board text removed: "Supervisor v1.0 altyr 2016"

Commit message: supervisior bugfixes final
Routing:
- net GND: track 160.2 -> 201.6 mm, vias 32 -> 40
- net (no net): track 14.0 -> 5.34 mm, vias 8 -> 3
- net SDA: track 142.2 -> 140.7 mm
- net SCL: track 88.5 -> 89.2 mm
Other:
- board outline added: 103.1 x 86.6 mm
